File: communication_board/communication_board.kicad_pcb (KiCad board)
At the start: 2 copper layers, 103 x 100 mm, 50 parts, among them J1 USB_IN, J2 IMU, J3 MINI_FUSE, J4 Motors, U1 FE1.1s, U2 FT232RL, U3 FT232RL, U4 MAX485E, Y1 Crystal

Commit message: mudancas finais
Parts:
- moved REF** 5.21 mm to (131.6, 40.1)
Changed lines of the file:
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@@
 			(outputformat 1)
 			(mirror no)
-			(drillshape 1)
+			(drillshape 0)
 			(scaleselection 1)
-			(outputdirectory "")
+			(outputdirectory "../gerber/")
 		)
 	)
@@
 		(tags "resistor")
 		(property "Reference" "R5"
-			(at 0 1.5 0)
+			(at 0 1.7315 0)
 			(layer "F.SilkS")
 			(effects
@@
 	(footprint "Humanoid:pcb_identification"
 		(layer "F.Cu")
-		(at 131.699 34.925)
+		(at 131.572 40.132)
 		(property "Reference" "REF**"
 			(at 0 -0.5 0)
@@
 		(tags "capacitor")
 		(property "Reference" "C8"
-			(at 0 1.5 0)
+			(at 0 1.7955 0)
 			(layer "F.SilkS")
 			(effects
@@
 		(tags "capacitor")
 		(property "Reference" "C7"
-			(at 0 1.65 0)
+			(at 0 1.8595 0)
 			(layer "F.SilkS")
 			(effects
@@
 	)
 	(gr_text "GND"
-		(at 187.9 99.5 90)
+		(at 187.9 99.695 90)
 		(layer "F.SilkS")
 		(effects
 			(font
-				(size 0.6 0.6)
-				(thickness 0.125)
+				(size 0.8 0.8)
+				(thickness 0.145)
 				(bold yes)
 			)
@@
 	)
 	(gr_text "VCC"
-		(at 187.9 91.7 90)
+		(at 187.9 91.948 90)
 		(layer "F.SilkS")
 		(effects
 			(font
-				(size 0.6 0.6)
-				(thickness 0.125)
+				(size 0.8 0.8)
+				(thickness 0.145)
 				(bold yes)
 			)
@@
 	)
 	(gr_text "D+"
-		(at 187.9 96.65 90)
+		(at 187.9 96.647 90)
 		(layer "F.SilkS")
 		(effects
 			(font
-				(size 0.6 0.6)
-				(thickness 0.125)
+				(size 0.8 0.8)
+				(thickness 0.145)
 				(bold yes)
 			)
@@
 	)
 	(gr_text "D-"
-		(at 187.9 94.1 90)
+		(at 187.9 94.234 90)
 		(layer "F.SilkS")
 		(effects
 			(font
-				(size 0.6 0.6)
-				(thickness 0.125)
+				(size 0.8 0.8)
+				(thickness 0.145)
 				(bold yes)
 			)
@@
 	)
 	(gr_text "JLCJLCJLCJLC"
-		(at 102.489 45.085 90)
+		(at 117.1956 93.726 0)
 		(layer "F.SilkS")
 		(effects
@@
 		(polygon
 			(pts
-				(xy 107.061 25.4) (xy 107.061 32.004) (xy 101.6 32.004) (xy 101.6 114.3) (xy 106.68 114.3) (xy 106.68 88.9)
-				(xy 137.16 88.9) (xy 137.16 121.92) (xy 193.04 121.92) (xy 193.04 88.9) (xy 200.66 88.9) (xy 200.66 31.75)
-				(xy 194.945 31.75) (xy 194.945 25.4)
+				(xy 151.892 85.852) (xy 107.061 85.852) (xy 101.6 85.852) (xy 101.6 114.3) (xy 106.68 114.3) (xy 106.68 88.9)
+				(xy 137.16 88.9) (xy 137.16 121.92) (xy 193.04 121.92) (xy 193.04 90.424) (xy 201.676 90.424) (xy 201.676 37.592)
+				(xy 163.576 37.592) (xy 163.576 74.676)
 			)
 		)
